File: element_foxtrot.kicad_pcb (KiCad board)
At the start: 4 copper layers, 202.5 x 307.5 mm, 147 parts, among them J1 Ext_Power, J2 Val**, J3 Val**, J4 Val**, J5 Program, J6 Conn_01x45, J7 USB, J8 Conn_01x45, P1 Val**, Q1 SQD40061EL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

Commit message: sync with library
Connections:
- P1 pad A8: (no net) -> Net-(P1-PadA8)
- P1 pad B8: (no net) -> Net-(P1-PadB8)
- SW1 pad 1: (no net) -> Net-(SW1-Pad1)
- SW1 pad 11: (no net) -> Net-(SW1-Pad11)
- SW1 pad 12: (no net) -> Net-(SW1-Pad12)
- SW1 pad 3: (no net) -> Net-(SW1-Pad3)
- SW1 pad 5: (no net) -> Net-(SW1-Pad5)
- SW1 pad 6: (no net) -> Net-(SW1-Pad6)
- SW1 pad 7: (no net) -> Net-(SW1-Pad7)
- SW1 pad 8: (no net) -> Net-(SW1-Pad8)
- U2 pad 11: (no net) -> /ATTACH
- U2 pad 14: (no net) -> Net-(U2-Pad14)
- U2 pad 17: (no net) -> Net-(U2-Pad17)
- U2 pad 3: (no net) -> Net-(U2-Pad3)
- U3 pad 6: (no net) -> Net-(U3-Pad6)
- U4 pad 3: (no net) -> Net-(U4-Pad3)
- U4 pad 6: (no net) -> Net-(U4-Pad6)
- U5 pad 2: (no net) -> Net-(U5-Pad2)
- U5 pad 6: (no net) -> Net-(U5-Pad6)
Other:
- board text added: "Module 3"
